File: kicad/het68-hat/het68-hat.kicad_sch (KiCad schematic)
At the start: 87 parts, among them J1 MIC1, J10 PWR, J11 PZ1, J12 PZ2, J13 PZ3, J14 PZ4, J17 UART, J2 MIC2, J3 MIC3, J4 MIC4, J5 MIC5, J6 MIC6, U1 Pico_Plus_2, U2 SN74LVC8T245, U3 SN74LVC8T245, U4 SN74LVC8T245, U5 AP2112K-1.8, U6 DRV8837C, U7 DPS310, U8 SHT40, U9 INA3221

Commit message: Ship a four-layer HAT that is fully routed and ready to fab.
GPIO for SD and LED move to the jack rows so firmware can follow PINOUT.csv; power and satellite boards stay as in v1.10.0.

Co-authored-by: Cursor <cursoragent@cursor.com>
Parts:
- removed R46: 10k, Resistor_SMD:R_0402_1005Metric, symbol Device:R
- added R50, R51, R52, R53, R54, R55: 100k, Resistor_SMD:R_0402_1005Metric, symbol Device:R
- J1, J2, J3, J4, J5, J6: footprint Connector_RJ:RJ45_Amphenol_RJHSE5380 -> het68:RJ45_RJHSE5380_het68
Connections:
- net +3V3: no longer U1.35 (ADC_VREF)
- net GND: now also R50.2, R51.2, R52.2, R53.2, R54.2, R55.2
- net LED1_G: now also U1.27 (GP21); no longer U1.14 (GP10)
- net LED2_G: now also U1.26 (GP20); no longer U1.15 (GP11)
- net LED3_G: now also U1.25 (GP19); no longer U1.16 (GP12)
- net LED4_G: now also U1.14 (GP10); no longer U1.17 (GP13)
- net LED5_G: now also U1.15 (GP11); no longer U1.19 (GP14)
- net LED6_G: now also U1.16 (GP12); no longer U1.29 (GP22)
- net SCK2_B: now also U2.19 (B3); no longer U2.20 (B2)
- net SCK3_B: now also U2.17 (B5); no longer U2.19 (B3)
- net SCK4_B: now also U3.17 (B5); no longer U2.18 (B4)
- net SCK5_B: now also U3.19 (B3); no longer U2.17 (B5)
- net SCK6_B: now also U3.21 (B1); no longer U2.16 (B6)
- net SCK_3V3: now also U3.3 (A1), U3.5 (A3), U3.7 (A5); no longer U2.4 (A2), U2.6 (A4), U2.8 (A6)
- net SD1_18: now also R50.1
- net SD1_3V3: now also U1.24 (GP18); no longer U1.21 (GP16)
- net SD2_18: now also R51.1
- net SD2_3V3: now also U1.22 (GP17); no longer U1.24 (GP18)
- net SD3_18: now also R52.1
- net SD3_3V3: now also U1.21 (GP16); no longer U1.26 (GP20)
- net SD4_18: now also U4.16 (B6), R53.1; no longer U4.18 (B4)
- net SD4_3V3: now also U1.17 (GP13), U4.8 (A6); no longer U1.31 (GP26), U4.6 (A4)
- net SD5_18: now also R54.1
- net SD5_3V3: now also U1.19 (GP14); no longer U1.32 (GP27)
- net SD6_18: now also U4.18 (B4), R55.1; no longer U4.16 (B6)
- net SD6_3V3: now also U1.20 (GP15), U4.6 (A4); no longer U1.34 (GP28), U4.8 (A6)
- net WS1_B: now also U2.20 (B2); no longer U3.21 (B1)
- net WS2_B: now also U2.18 (B4); no longer U3.20 (B2)
- net WS3_B: now also U2.16 (B6); no longer U3.19 (B3)
- net WS4_B: now also U3.16 (B6); no longer U3.18 (B4)
- net WS5_B: now also U3.18 (B4); no longer U3.17 (B5)
- net WS6_B: now also U3.20 (B2); no longer U3.16 (B6)
- net WS_3V3: now also U2.4 (A2), U2.6 (A4), U2.8 (A6); no longer U3.3 (A1), U3.5 (A3), U3.7 (A5)
- net RUN: no longer names the net of U1.30 (RUN)
- no-connect marks 17 -> 19

Commit message: Fit every board on printed.cz prototype: 2-layer, 0603, ENIG.
HAT is 140×140 mm so it routes on two layers without 0402 or BGA; satellite and power use the same stack, drill and finish.

Co-authored-by: Cursor <cursoragent@cursor.com>
Parts:
- C1, C13, C2: footprint Capacitor_SMD:C_0402_1005Metric -> Capacitor_SMD:C_0603_1608Metric; MPN CL05A105KA5NQNC -> CL10A105KA8NNNC
- C10, C11, C12, C14, C5, C6, C7, C8, C9: footprint Capacitor_SMD:C_0402_1005Metric -> Capacitor_SMD:C_0603_1608Metric; MPN CL05B104KB5NNNC -> CL10B104KB8NNNC
- R10, R11, R13, R14, R16, R17, R19, R20, R22, R23, R25, R26: footprint Resistor_SMD:R_0402_1005Metric -> Resistor_SMD:R_0603_1608Metric; MPN RC0402FR-0733RL -> RC0603FR-0733RL
- R12, R15, R18, R21, R24, R27: footprint Resistor_SMD:R_0402_1005Metric -> Resistor_SMD:R_0603_1608Metric; MPN RC0402FR-07100RL -> RC0603FR-07100RL
- R42, R43, R44, R45: footprint Resistor_SMD:R_0402_1005Metric -> Resistor_SMD:R_0603_1608Metric; MPN RC0402FR-074K7L -> RC0603FR-074K7L
- R50, R51, R52, R53, R54, R55: footprint Resistor_SMD:R_0402_1005Metric -> Resistor_SMD:R_0603_1608Metric; MPN RC0402FR-07100KL -> RC0603FR-07100KL
