File: kicad/het68-pwr/het68-pwr.kicad_sch (KiCad schematic)
At the start: 19 parts, among them J1 AC_IN, J2 USB_C, J3 VSYS_OUT

Commit message: Switch the boards to two layers and specify the power sources.
The HAT is no longer four-layer and the gerbers match that stackup. The power board now names the clamp CT, solar MPPT, 21700 cell and 5 V output; those charger parts are not drawn in KiCad yet.

Co-authored-by: Cursor <cursoragent@cursor.com>
Parts:
- added R4: 100, Resistor_SMD:R_1206_3216Metric, symbol Device:R
Connections:
- net AC1: now also R4.1
- net AC2: now also R4.2

Commit message: Protect the CT secondary and ship clean power and satellite fab files.
Add burden, LC filter and crowbar on the power board, close DRC on power and satellite, and refresh the board previews for v1.10.0.

Co-authored-by: Cursor <cursoragent@cursor.com>
Parts:
- added C4: 1u/100V, Capacitor_SMD:C_1206_3216Metric, symbol Device:C
- added L1: 470uH, Inductor_THT:L_Radial_D10.0mm_P5.00mm_Fastron_07P, symbol Device:L
- added Q1: X0202MN, Package_TO_SOT_SMD:SOT-223, symbol Triac_Thyristor:X0202MN
- added R5: 1k, Resistor_SMD:R_0805_2012Metric, symbol Device:R
- C1: value 470u/25V -> 470u/50V; MPN electrolytic 470u 25V -> electrolytic 470u 50V
- D5: value SMBJ15A -> BZX84-C24; footprint Diode_SMD:D_SMB -> Diode_SMD:D_SOD-323; MPN SMBJ15A -> BZX84-C24
- J1: MPN sekundar split-core, NE sit 230 V -> sekundar CT / split-core, NE sit 230 V ani 22 kV
- R4: footprint Resistor_SMD:R_1206_3216Metric -> Resistor_THT:R_Axial_DIN0207_L6.3mm_D2.5mm_P10.16mm_Horizontal; MPN RC1206FR-07100RL -> 100R THT burden
Connections:
- net AC1: now also L1.1; no longer F1.1
- net AC2: now also C4.2
- net DC: now also Q1.2 (A), Q1.4 (A), R5.1; no longer D5.1 (K)
- net GND: now also Q1.1 (K)
- new net AC1L: C4.1, F1.1, L1.2
- new net SCR_G: D5.1 (K), Q1.3 (G), R5.2
Other:
- title: het68 napajeni — jen sekundar split-core -> het68 napajeni — sekundar CT, burden, LC, crowbar

Commit message: Fit every board on printed.cz prototype: 2-layer, 0603, ENIG.
HAT is 140×140 mm so it routes on two layers without 0402 or BGA; satellite and power use the same stack, drill and finish.

Co-authored-by: Cursor <cursoragent@cursor.com>
Parts:
- R1, R2: footprint Resistor_SMD:R_0402_1005Metric -> Resistor_SMD:R_0603_1608Metric; MPN RC0402FR-075K1L -> RC0603FR-075K1L
- R3: footprint Resistor_SMD:R_0402_1005Metric -> Resistor_SMD:R_0603_1608Metric; MPN RC0402FR-072K2L -> RC0603FR-072K2L
