File: kicad/het68-core/het68-core.kicad_pcb (KiCad board)
At the start: 6 copper layers, 160 x 100 mm, 134 parts, among them J1 MIC1, J11 PZ1, J12 PZ2, J13 PZ3, J14 PZ4, J2 MIC2, J3 MIC3, J4 MIC4, J5 MIC5, J6 MIC6, U1 RP2350B, U10 SN65LVDS047, U11 SN65LVDS047, U12 SN65LVDS047, U13 SN65LVDS32, U14 SN65LVDS32, U2 W25Q128JVSIQ, U3 APS6404L, U4 AP2112K-3.3, U5 AP2112K-1.8, U6 DRV8837C, U7 DPS310, U8 SHT40, U9 ADXL355, Y1 12MHz

Commit message: Ship the furthest routed v4 boards with matching previews.
The satellite signal nets are closed, the five boards have no shorts, and the gerbers and renders follow this copper.

Co-authored-by: Cursor <cursoragent@cursor.com>
Parts:
- moved H1 65.0 mm to (4.95, 71.0)
Connections:
- D_STAT pad 2: unconnected-(D_STAT-DOUT-Pad2) -> (no net)
- J_MESH pad 8: unconnected-(J_MESH-8-Pad8) -> (no net)
- J_STAMP pad 8: unconnected-(J_STAMP-8-Pad8) -> (no net)
- J_USB pad A6: unconnected-(J_USB-D+-PadA6) -> (no net)
- J_USB pad A7: unconnected-(J_USB-D--PadA7) -> (no net)
- J_USB pad A8: unconnected-(J_USB-SBU1-PadA8) -> (no net)
- J_USB pad B6: unconnected-(J_USB-D+-PadB6) -> (no net)
- J_USB pad B7: unconnected-(J_USB-D--PadB7) -> (no net)
- J_USB pad B8: unconnected-(J_USB-SBU2-PadB8) -> (no net)
- U1 pad 48: unconnected-(U1-GPIO39-Pad48) -> (no net)
- U1 pad 49: unconnected-(U1-GPIO40-Pad49) -> (no net)
- U1 pad 52: unconnected-(U1-GPIO41-Pad52) -> (no net)
- U1 pad 53: unconnected-(U1-GPIO42-Pad53) -> (no net)
- U1 pad 54: unconnected-(U1-GPIO43-Pad54) -> (no net)
- U1 pad 55: unconnected-(U1-GPIO44-Pad55) -> (no net)
- U1 pad 56: unconnected-(U1-GPIO45-Pad56) -> (no net)
- U1 pad 57: unconnected-(U1-GPIO46-Pad57) -> (no net)
- U1 pad 58: unconnected-(U1-GPIO47-Pad58) -> (no net)
- U14 pad 11: unconnected-(U14-3Y-Pad11) -> (no net)
- U14 pad 13: unconnected-(U14-4Y-Pad13) -> (no net)
- U4 pad 4: unconnected-(U4-NC-Pad4) -> (no net)
- U5 pad 4: unconnected-(U5-NC-Pad4) -> (no net)
- U9 pad 1: unconnected-(U9-NC1-Pad1) -> (no net)
- U9 pad 10: unconnected-(U9-NC10-Pad10) -> (no net)
- U9 pad 15: unconnected-(U9-NC15-Pad15) -> (no net)
- U9 pad 16: unconnected-(U9-NC16-Pad16) -> (no net)
- U9 pad 3: unconnected-(U9-NC3-Pad3) -> (no net)
- U9 pad 8: unconnected-(U9-INT2-Pad8) -> (no net)
- U9 pad 9: unconnected-(U9-INT1-Pad9) -> (no net)
Routing:
- net +3V3_DIG: track 1193.4 -> 1831.7 mm, vias 140 -> 164
- net +5V_ALWAYS: track 237.8 -> 434.1 mm, vias 14 -> 20
- net GND: track 580.9 -> 663.1 mm, vias 351 -> 361
- net I2S_SCK: track 277.6 -> 325.0 mm, vias 20 -> 22
- net WS5_N: track 16.2 -> 60.6 mm, vias 1 -> 3
- net WS5_PJ: track 49.7 -> 92.4 mm, vias 2 -> 4
- net WS5_P: track 10.7 -> 52.4 mm, vias 1 -> 3
- net WS3_PJ: track 42.0 -> 75.1 mm, vias 1 -> 4
- net PIEZO_P: track 63.5 -> 87.5 mm
- net +1V8_AUDIO: track 306.9 -> 325.7 mm
- net DSP_AWAKE: track 106.7 -> 118.0 mm, vias 8 -> 9
- net WS2_PJ: track 89.2 -> 99.2 mm, vias 3 -> 5
- net I2C1_SDA: track 174.8 -> 184.4 mm
- net I2C1_SCL: track 143.5 -> 135.0 mm
- net RUN: track 336.2 -> 344.2 mm
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