File: kicad/het68-core/het68-core.kicad_pcb (KiCad board)
At the start: 6 copper layers, 160 x 100 mm, 134 parts, among them J1 MIC1, J11 PZ1, J12 PZ2, J13 PZ3, J14 PZ4, J2 MIC2, J3 MIC3, J4 MIC4, J5 MIC5, J6 MIC6, U1 RP2350B, U10 SN65LVDS047, U11 SN65LVDS047, U12 SN65LVDS047, U13 SN65LVDS32, U14 SN65LVDS32, U2 W25Q128JVSIQ, U3 APS6404L, U4 AP2112K-3.3, U5 AP2112K-1.8, U6 DRV8837C, U7 DPS310, U8 SHT40, U9 ADXL355, Y1 12MHz

Commit message: Stand the RJ45 plugs upright and show the mode shunt.
The core and satellite jacks are a vertical 8P8C. The plug axis leaves
the board face instead of running off the edge. The docs and the v480
renders include the satellite mode headers. DRC has no shorts. Some
jack pins, and the tracks the new pad grid cut, are still open.

Co-authored-by: fedurca <fedurca@users.noreply.github.com>
Parts:
- J1, J2, J3, J4, J5, J6: footprint het68:RJ45_RJHSE5380_het68 -> het68:RJ45_Vertical_het68
- moved J1 2.80 mm to (14.0, 7.20)
- moved J2 2.80 mm to (38.0, 7.20)
- moved J3 2.80 mm to (62.0, 7.20)
- moved J4 2.80 mm to (86.0, 7.20)
- moved J5 2.80 mm to (110.0, 7.20)
- moved J6 2.80 mm to (134.0, 7.20)
Routing:
- net I2C1_SDA: track 226.6 -> 184.7 mm
- net WS2_N: track 154.9 -> 120.9 mm
- net WS2_P: track 142.2 -> 110.6 mm
- net SD2_P: track 387.6 -> 358.2 mm
- net MIC5_3V3: track 27.5 -> 51.5 mm
- net SCK2_P: track 139.0 -> 116.3 mm
- net SCK4_NJ: track 23.5 -> 43.2 mm
- net SCK3_NJ: track 23.5 -> 43.2 mm
- net SD4_NJ: track 37.3 -> 53.4 mm
- net SD2_NJ: track 34.6 -> 50.5 mm
- net MIC2_3V3: track 28.3 -> 44.0 mm
- net MIC6_3V3: track 31.1 -> 45.1 mm
- net SD4_PJ: track 36.8 -> 48.5 mm
- net WS4_NJ: track 22.6 -> 34.3 mm
- net SD6_PJ: track 45.4 -> 56.9 mm
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