File: kicad/het68-core/het68-core.kicad_sch (KiCad schematic)
At the start: 103 parts, among them J1 MIC1, J11 PZ1, J12 PZ2, J13 PZ3, J14 PZ4, J2 MIC2, J3 MIC3, J4 MIC4, J5 MIC5, J6 MIC6, U1 RP2350B, U10 SN65LVDS047, U11 SN65LVDS047, U12 SN65LVDS047, U13 SN65LVDS32, U14 SN65LVDS32, U2 W25Q128JVSIQ, U3 APS6404L, U4 AP2112K-3.3, U5 AP2112K-1.8, U6 DRV8837C, U7 DPS310, U8 SHT40, U9 ADXL355, Y1 12MHz

Commit message: Ship v4.1.0 as a Core+satellite+power kit without the v3 HAT.
LVDS now has 100 ohm receivers, SD common-mode chokes, and 3V3 ferrites for a noisy line; the kit BOM and 3D previews match that schematic.

Co-authored-by: Cursor <cursoragent@cursor.com>
Parts:
- added FB1, FB2, FB3, FB4, FB5, FB6: 600R, Inductor_SMD:L_0603_1608Metric, symbol Device:FerriteBead
- added FL1C, FL2C, FL3C, FL4C, FL5C, FL6C: CMC, Inductor_SMD:L_CommonModeChoke_Coilank_ACM2012, symbol het68:CMC
- added R_I2S_SCK, R_I2S_WS: 33, Resistor_SMD:R_0603_1608Metric, symbol Device:R
- added R_SD1, R_SD2, R_SD3, R_SD4, R_SD5, R_SD6: 100, Resistor_SMD:R_0603_1608Metric, symbol Device:R
- C_X1, C_X2: MPN CL10B104KB8NNNC -> CL10C150JB8NNNC
- R_RX, R_TX: MPN RC0603FR-0733RL -> RC0603FR-0722RL
Connections:
- net I2S_SCK: now also R_I2S_SCK.2; no longer U1.7 (GPIO9)
- net I2S_WS: now also R_I2S_WS.2; no longer U1.6 (GPIO8)
- net MIC1_3V3: now also FB1.2; no longer F1.2
- net MIC2_3V3: now also FB2.2; no longer F2.2
- net MIC3_3V3: now also FB3.2; no longer F3.2
- net MIC4_3V3: now also FB4.2; no longer F4.2
- net MIC5_3V3: now also FB5.2; no longer F5.2
- net MIC6_3V3: now also FB6.2; no longer F6.2
- net SD1_N: now also FL1C.2, R_SD1.2
- net SD1_NJ: now also FL1C.3
- net SD1_P: now also FL1C.1, R_SD1.1
- net SD1_PJ: now also FL1C.4
- net SD2_N: now also FL2C.2, R_SD2.2
- net SD2_NJ: now also FL2C.3
- net SD2_P: now also FL2C.1, R_SD2.1
- net SD2_PJ: now also FL2C.4
- net SD3_N: now also FL3C.2, R_SD3.2
- net SD3_NJ: now also FL3C.3
- net SD3_P: now also FL3C.1, R_SD3.1
- net SD3_PJ: now also FL3C.4
- net SD4_N: now also FL4C.2, R_SD4.2
- net SD4_NJ: now also FL4C.3
- net SD4_P: now also FL4C.1, R_SD4.1
- net SD4_PJ: now also FL4C.4
- net SD5_N: now also FL5C.2, R_SD5.2
- net SD5_NJ: now also FL5C.3
- net SD5_P: now also FL5C.1, R_SD5.1
- net SD5_PJ: now also FL5C.4
- net SD6_N: now also FL6C.2, R_SD6.2
- net SD6_NJ: now also FL6C.3
- net SD6_P: now also FL6C.1, R_SD6.1
- net SD6_PJ: now also FL6C.4
- new net I2S_SCK_MCU: R_I2S_SCK.1, U1.7 (GPIO9)
- new net I2S_WS_MCU: R_I2S_WS.1, U1.6 (GPIO8)
- new net MIC1_FB: F1.2, FB1.1
- new net MIC2_FB: F2.2, FB2.1
- new net MIC3_FB: F3.2, FB3.1
- new net MIC4_FB: F4.2, FB4.1
- new net MIC5_FB: F5.2, FB5.1
- new net MIC6_FB: F6.2, FB6.1

Commit message: Add a Core status LED and three buttons, and fit a 21700 holder.
RESET, BOOT and USER sit on the east edge with one SK6812; the power board uses a Keystone 1122 instead of an 18650 sled. Masks, schematics and JLCPCB gerber zips are in the tree.

Co-authored-by: Cursor <cursoragent@cursor.com>
Parts:
- added C_STAT: 100n, Capacitor_SMD:C_0603_1608Metric, symbol Device:C
- added D_STAT: SK6812, LED_SMD:LED_WS2812B_PLCC4_5.0x5.0mm_P3.2mm, symbol LED:WS2812B
- added R_CS, R_USR: 10k, Resistor_SMD:R_0603_1608Metric, symbol Device:R
- added SW_BOOT: BOOT, Button_Switch_SMD:SW_SPST_PTS645Sx43SMTR92, symbol Switch:SW_Push
- added SW_RST: RESET, Button_Switch_SMD:SW_SPST_PTS645Sx43SMTR92, symbol Switch:SW_Push
- added SW_USR: USER, Button_Switch_SMD:SW_SPST_PTS645Sx43SMTR92, symbol Switch:SW_Push
Connections:
- net +3V3_DIG: now also C18A.2, C18B.2, C3V3A.2, C3V3B.2, C_ADX.2, C_DVDD.2, C_IO1.2, C_IO2.2, C_IO3.2, C_LV1.2, C_LV2.2, C_LV3.2, C_PZ.2, C_RX1.2, C_RX2.2, C_VBUS.2, C_X1.2, C_X2.2, D_RX.2 (A2), D_TX.2 (A2), J1.SH (SHIELD), J2.SH (SHIELD), J3.SH (SHIELD), J4.SH (SHIELD), J5.SH (SHIELD), J6.SH (SHIELD), J_MESH.1, J_PWR.19, J_PWR.2, J_PWR.20, J_PWR.4, J_PWR.6, J_STAMP.1, J_SWD.2, J_USB.A1 (GND), J_USB.A12 (GND), J_USB.B1 (GND), J_USB.B12 (GND), J_USB.SH (SHIELD), R_CC1.2, R_CC2.2, R_SH.2, R_WK.2, U1.62 (VREG_PGND), U1.81 (GND), U10.16 (ENn), U10.7 (GND), U11.16 (ENn), U11.7 (GND), U12.16 (ENn), U12.7 (GND), U13.12 (Gn), U13.8 (GND), U14.10 (3A), U14.12 (Gn), U14.14 (4A), U14.15 (4B), U14.8 (GND), U14.9 (3B), U2.4 (GND), U3.4 (GND), U4.2 (GND), U5.2 (GND), U6.4 (GND), U6.9 (GND), U7.1 (GND), U7.7 (GND), U8.4 (VSS), U9.17 (EP), U9.4 (GND), U9.5 (GND2), U9.7 (AUX), Y1.2 (GND1), Y1.4 (GND2), C_STAT.1, C_STAT.2, D_STAT.1 (VDD), D_STAT.3 (VSS), R_CS.2, R_USR.2, SW_BOOT.2, SW_RST.2, SW_USR.2
- net QSPI_SS: now also R_CS.1, SW_BOOT.1
- net RUN: now also SW_RST.1
- net STATUS_DIN: now reaches U1.46 (GPIO37)
- net STATUS_DIN: now also D_STAT.4 (DIN)
- net BTN_USER: now reaches U1.47 (GPIO38)
- net BTN_USER: now also R_USR.1, SW_USR.1
- removed net GND: C18A.2, C18B.2, C3V3A.2, C3V3B.2, C_ADX.2, C_DVDD.2, C_IO1.2, C_IO2.2, C_IO3.2, C_LV1.2, C_LV2.2, C_LV3.2, C_PZ.2, C_RX1.2, C_RX2.2, C_VBUS.2, C_X1.2, C_X2.2, D_RX.2 (A2), D_TX.2 (A2), J1.SH (SHIELD), J2.SH (SHIELD), J3.SH (SHIELD), J4.SH (SHIELD), J5.SH (SHIELD), J6.SH (SHIELD), J_MESH.1, J_MESH.5, J_PWR.19, J_PWR.2, J_PWR.20, J_PWR.4, J_PWR.6, J_STAMP.1, J_STAMP.5, J_SWD.2, J_USB.A1 (GND), J_USB.A12 (GND), J_USB.B1 (GND), J_USB.B12 (GND), J_USB.SH (SHIELD), R_CC1.2, R_CC2.2, R_SH.2, R_WK.1, R_WK.2, U1.62 (VREG_PGND), U1.81 (GND), U10.16 (ENn), U10.7 (GND), U11.16 (ENn), U11.7 (GND), U12.16 (ENn), U12.7 (GND), U13.12 (Gn), U13.8 (GND), U14.10 (3A), U14.12 (Gn), U14.14 (4A), U14.15 (4B), U14.8 (GND), U14.9 (3B), U2.4 (GND), U3.4 (GND), U4.2 (GND), U4.3 (EN), U5.2 (GND), U5.3 (EN), U6.4 (GND), U6.9 (GND), U7.1 (GND), U7.7 (GND), U8.4 (VSS), U9.17 (EP), U9.4 (GND), U9.5 (GND2), U9.7 (AUX), Y1.2 (GND1), Y1.4 (GND2)
- new net WAKE_DSP: J_MESH.5, J_STAMP.5, R_WK.1, U4.3 (EN), U5.3 (EN)
- no-connect marks 30 -> 29
