File: kicad/het68-core/het68-core.kicad_sch (KiCad schematic)
At the start: 130 parts, among them J1 MIC1, J11 PZ1, J12 PZ2, J13 PZ3, J14 PZ4, J2 MIC2, J3 MIC3, J4 MIC4, J5 MIC5, J6 MIC6, U1 RP2350B, U10 SN65LVDS047, U11 SN65LVDS047, U12 SN65LVDS047, U13 SN65LVDS32, U14 SN65LVDS32, U2 W25Q128JVSIQ, U3 APS6404L, U4 AP2112K-3.3, U5 AP2112K-1.8, U6 DRV8837C, U7 DPS310, U8 SHT40, U9 ADXL355, Y1 12MHz

Commit message: Stand the RJ45 plugs upright and show the mode shunt.
The core and satellite jacks are a vertical 8P8C. The plug axis leaves
the board face instead of running off the edge. The docs and the v480
renders include the satellite mode headers. DRC has no shorts. Some
jack pins, and the tracks the new pad grid cut, are still open.

Co-authored-by: fedurca <fedurca@users.noreply.github.com>
Parts:
- J1, J2, J3, J4, J5, J6: footprint het68:RJ45_RJHSE5380_het68 -> het68:RJ45_Vertical_het68; MPN RJHSE-5380 -> RJ45-8P8C-VERT
Changed lines of the file:
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@@
     (property "Reference" "J1" (at 400.0 407.36 0) (effects (font (size 1.27 1.27))))
     (property "Value" "MIC1" (at 400.0 403.36 0) (effects (font (size 1.27 1.27))))
-    (property "Footprint" "het68:RJ45_RJHSE5380_het68" (at 400.0 405.36 0) (effects (font (size 1.27 1.27)) (hide yes)))
+    (property "Footprint" "het68:RJ45_Vertical_het68" (at 400.0 405.36 0) (effects (font (size 1.27 1.27)) (hide yes)))
     (property "Datasheet" "" (at 400.0 405.36 0) (effects (font (size 1.27 1.27)) (hide yes)))
-    (property "MPN" "RJHSE-5380" (at 400.0 405.36 0) (effects (font (size 1.27 1.27)) (hide yes)))
+    (property "MPN" "RJ45-8P8C-VERT" (at 400.0 405.36 0) (effects (font (size 1.27 1.27)) (hide yes)))
     (pin "1")
     (pin "2")
@@
     (property "Reference" "J2" (at 400.0 176.56 0) (effects (font (size 1.27 1.27))))
     (property "Value" "MIC2" (at 400.0 172.56 0) (effects (font (size 1.27 1.27))))
-    (property "Footprint" "het68:RJ45_RJHSE5380_het68" (at 400.0 174.56 0) (effects (font (size 1.27 1.27)) (hide yes)))
+    (property "Footprint" "het68:RJ45_Vertical_het68" (at 400.0 174.56 0) (effects (font (size 1.27 1.27)) (hide yes)))
     (property "Datasheet" "" (at 400.0 174.56 0) (effects (font (size 1.27 1.27)) (hide yes)))
-    (property "MPN" "RJHSE-5380" (at 400.0 174.56 0) (effects (font (size 1.27 1.27)) (hide yes)))
+    (property "MPN" "RJ45-8P8C-VERT" (at 400.0 174.56 0) (effects (font (size 1.27 1.27)) (hide yes)))
     (pin "1")
     (pin "2")
@@
     (property "Reference" "J3" (at 490.0 425.14 0) (effects (font (size 1.27 1.27))))
     (property "Value" "MIC3" (at 490.0 421.14 0) (effects (font (size 1.27 1.27))))
-    (property "Footprint" "het68:RJ45_RJHSE5380_het68" (at 490.0 423.14 0) (effects (font (size 1.27 1.27)) (hide yes)))
+    (property "Footprint" "het68:RJ45_Vertical_het68" (at 490.0 423.14 0) (effects (font (size 1.27 1.27)) (hide yes)))
     (property "Datasheet" "" (at 490.0 423.14 0) (effects (font (size 1.27 1.27)) (hide yes)))
-    (property "MPN" "RJHSE-5380" (at 490.0 423.14 0) (effects (font (size 1.27 1.27)) (hide yes)))
+    (property "MPN" "RJ45-8P8C-VERT" (at 490.0 423.14 0) (effects (font (size 1.27 1.27)) (hide yes)))
     (pin "1")
     (pin "2")
@@
     (property "Reference" "J4" (at 490.0 194.34000000000003 0) (effects (font (size 1.27 1.27))))
     (property "Value" "MIC4" (at 490.0 190.34000000000003 0) (effects (font (size 1.27 1.27))))
-    (property "Footprint" "het68:RJ45_RJHSE5380_het68" (at 490.0 192.34000000000003 0) (effects (font (size 1.27 1.27)) (hide yes)))
+    (property "Footprint" "het68:RJ45_Vertical_het68" (at 490.0 192.34000000000003 0) (effects (font (size 1.27 1.27)) (hide yes)))
     (property "Datasheet" "" (at 490.0 192.34000000000003 0) (effects (font (size 1.27 1.27)) (hide yes)))
-    (property "MPN" "RJHSE-5380" (at 490.0 192.34000000000003 0) (effects (font (size 1.27 1.27)) (hide yes)))
+    (property "MPN" "RJ45-8P8C-VERT" (at 490.0 192.34000000000003 0) (effects (font (size 1.27 1.27)) (hide yes)))
     (pin "1")
     (pin "2")
@@
     (property "Reference" "J5" (at 580.0 425.14 0) (effects (font (size 1.27 1.27))))
     (property "Value" "MIC5" (at 580.0 421.14 0) (effects (font (size 1.27 1.27))))
-    (property "Footprint" "het68:RJ45_RJHSE5380_het68" (at 580.0 423.14 0) (effects (font (size 1.27 1.27)) (hide yes)))
+    (property "Footprint" "het68:RJ45_Vertical_het68" (at 580.0 423.14 0) (effects (font (size 1.27 1.27)) (hide yes)))
     (property "Datasheet" "" (at 580.0 423.14 0) (effects (font (size 1.27 1.27)) (hide yes)))
-    (property "MPN" "RJHSE-5380" (at 580.0 423.14 0) (effects (font (size 1.27 1.27)) (hide yes)))
+    (property "MPN" "RJ45-8P8C-VERT" (at 580.0 423.14 0) (effects (font (size 1.27 1.27)) (hide yes)))
     (pin "1")
     (pin "2")
@@
     (property "Reference" "J6" (at 580.0 194.34000000000003 0) (effects (font (size 1.27 1.27))))
     (property "Value" "MIC6" (at 580.0 190.34000000000003 0) (effects (font (size 1.27 1.27))))
-    (property "Footprint" "het68:RJ45_RJHSE5380_het68" (at 580.0 192.34000000000003 0) (effects (font (size 1.27 1.27)) (hide yes)))
+    (property "Footprint" "het68:RJ45_Vertical_het68" (at 580.0 192.34000000000003 0) (effects (font (size 1.27 1.27)) (hide yes)))
     (property "Datasheet" "" (at 580.0 192.34000000000003 0) (effects (font (size 1.27 1.27)) (hide yes)))
-    (property "MPN" "RJHSE-5380" (at 580.0 192.34000000000003 0) (effects (font (size 1.27 1.27)) (hide yes)))
-    (pin "1")
-    (pin "2")
+    (property "MPN" "RJ45-8P8C-VERT" (at 580.0 192.34000000000003 0) (effects (font (size 1.27 1.27)) (hide yes)))
+    (pin "1")
+    (pin "2")
