File: kicad/het68-pwr-vvn/het68-pwr-vvn.kicad_sch (KiCad schematic)
At the start: 60 parts, among them J1 CT_SEC, J2 USB_C, J3 VOUT, Q1 X0202MN

Commit message: Add a Core status LED and three buttons, and fit a 21700 holder.
RESET, BOOT and USER sit on the east edge with one SK6812; the power board uses a Keystone 1122 instead of an 18650 sled. Masks, schematics and JLCPCB gerber zips are in the tree.

Co-authored-by: Cursor <cursoragent@cursor.com>
Parts:
- BT1: value LiFePO4_1S -> 21700; footprint Battery:BatteryHolder_Keystone_1042_1x18650 -> het68:Keystone_1122_21700; MPN LiFePO4 / LTO 1S -> Keystone 1122
