File: kicad/het68-sat/het68-sat.kicad_sch (KiCad schematic)
At the start: 36 parts, among them J1 RJ45, U1 AP2112K-1.8, U2 SN65LVDS2, U3 SN65LVDS2, U4 SN65LVDS1, U5 TXS0104E

Commit message: Ship v4.1.0 as a Core+satellite+power kit without the v3 HAT.
LVDS now has 100 ohm receivers, SD common-mode chokes, and 3V3 ferrites for a noisy line; the kit BOM and 3D previews match that schematic.

Co-authored-by: Cursor <cursoragent@cursor.com>
Parts:
- added FB1: 600R, Inductor_SMD:L_0603_1608Metric, symbol Device:FerriteBead
- added R_SCK, R_WS: 100, Resistor_SMD:R_0603_1608Metric, symbol Device:R
Connections:
- net +3V3: now also FB1.2; no longer F1.2
- net SCK_N: now also R_SCK.2
- net SCK_P: now also R_SCK.1
- net WS_N: now also R_WS.2
- net WS_P: now also R_WS.1
- new net +3V3_FB: F1.2, FB1.1
