File: kicad/het68-sat/het68-sat.kicad_sch (KiCad schematic)
At the start: 39 parts, among them J1 RJ45, U1 AP2112K-1.8, U2 SN65LVDS2, U3 SN65LVDS2, U4 SN65LVDS1, U5 TXS0104E

Commit message: Select the satellite link mode with a shunt on the board.
The cable has no spare wire, so each of SCK, WS and SD uses a 2x3 header. One horizontal shunt picks the row: north is LVDS, middle is 3.3 V through the translator, south is 1.8 V on the T5848. The microphone supply stays 1.8 V and the RJ45 shield is grounded.

DRC reports no shorts. Airwires remain on OE, a short SD_3V3 gap at U5, WS_LVDS, WS_P, WS_T and WS_N.

Co-authored-by: fedurca <fedurca@users.noreply.github.com>
Parts:
- added JP_OE: OE, Connector_PinHeader_2.54mm:PinHeader_1x02_P2.54mm_Vertical, symbol het68:Conn_1x02
- added JP_SCK, JP_SD, JP_WS: MODE, Connector_PinHeader_2.54mm:PinHeader_2x03_P2.54mm_Vertical, symbol het68:Conn_2x03
- added JP_SDN: SDN, Connector_PinHeader_2.54mm:PinHeader_1x03_P2.54mm_Vertical, symbol het68:Conn_1x03
- added JP_TSCK, JP_TWS: T, Connector_PinHeader_2.54mm:PinHeader_1x02_P2.54mm_Vertical, symbol het68:Conn_1x02
- added R_OE: 10k, Resistor_SMD:R_0603_1608Metric, symbol Device:R
- added R_SD3: 100k, Resistor_SMD:R_0603_1608Metric, symbol Device:R
Connections:
- net +3V3: now also R_OE.1; no longer U5.8 (OE)
- net GND: now also J1.SH (SHIELD), JP_OE.1, JP_SDN.3, R_SD3.2
- net SCK: now also JP_SCK.6
- net SCK_3V3: now also JP_SCK.2, JP_SCK.4; no longer U2.5 (ROUT)
- net SCK_N: now also JP_TSCK.2; no longer R_SCK.2
- net SCK_P: now also JP_SCK.3, JP_SCK.5
- net SD: now also JP_SD.5
- net SD_3V3: now also JP_SD.3, R_SD3.1
- net SD_N: now also JP_SDN.2; no longer U4.4 (Z)
- net SD_P: now also JP_SD.2, JP_SD.4, JP_SD.6; no longer U4.3 (Y)
- net WS: now also JP_WS.6
- net WS_3V3: now also JP_WS.2, JP_WS.4; no longer U3.5 (ROUT)
- net WS_N: now also JP_TWS.2; no longer R_WS.2
- net WS_P: now also JP_WS.3, JP_WS.5
- new net OE: JP_OE.2, R_OE.2, U5.8 (OE)
- new net SCK_LVDS: JP_SCK.1, U2.5 (ROUT)
- new net SCK_T: JP_TSCK.1, R_SCK.2
- new net SD_Y: JP_SD.1, U4.3 (Y)
- new net SD_Z: JP_SDN.1, U4.4 (Z)
- new net WS_LVDS: JP_WS.1, U3.5 (ROUT)
- new net WS_T: JP_TWS.1, R_WS.2
- no-connect marks 9 -> 8
Other:
- title: het68 satelit 6L LVDS + T5848 + 8x SK6812 -> het68 satelit 6L — režim linky propojkou

Commit message: Stand the RJ45 plugs upright and show the mode shunt.
The core and satellite jacks are a vertical 8P8C. The plug axis leaves
the board face instead of running off the edge. The docs and the v480
renders include the satellite mode headers. DRC has no shorts. Some
jack pins, and the tracks the new pad grid cut, are still open.

Co-authored-by: fedurca <fedurca@users.noreply.github.com>
Parts:
- J1: footprint het68:RJ45_RJHSE5380_het68 -> het68:RJ45_Vertical_het68; MPN RJHSE-5380 -> RJ45-8P8C-VERT
Changed lines of the file:
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@@
     (property "Reference" "J1" (at 40.0 502.0 0) (effects (font (size 1.27 1.27))))
     (property "Value" "RJ45" (at 40.0 498.0 0) (effects (font (size 1.27 1.27))))
-    (property "Footprint" "het68:RJ45_RJHSE5380_het68" (at 40.0 500.0 0) (effects (font (size 1.27 1.27)) (hide yes)))
+    (property "Footprint" "het68:RJ45_Vertical_het68" (at 40.0 500.0 0) (effects (font (size 1.27 1.27)) (hide yes)))
     (property "Datasheet" "" (at 40.0 500.0 0) (effects (font (size 1.27 1.27)) (hide yes)))
-    (property "MPN" "RJHSE-5380" (at 40.0 500.0 0) (effects (font (size 1.27 1.27)) (hide yes)))
+    (property "MPN" "RJ45-8P8C-VERT" (at 40.0 500.0 0) (effects (font (size 1.27 1.27)) (hide yes)))
     (pin "1")
     (pin "2")
