File: kicad/het68-sat/het68-sat.kicad_pcb (KiCad board)
At the start: 6 copper layers, 50 x 80 mm, 43 parts, among them J1 RJ45, U1 AP2112K-1.8, U2 SN65LVDS2, U3 SN65LVDS2, U4 SN65LVDS1, U5 TXS0104E

Commit message: Select the satellite link mode with a shunt on the board.
The cable has no spare wire, so each of SCK, WS and SD uses a 2x3 header. One horizontal shunt picks the row: north is LVDS, middle is 3.3 V through the translator, south is 1.8 V on the T5848. The microphone supply stays 1.8 V and the RJ45 shield is grounded.

DRC reports no shorts. Airwires remain on OE, a short SD_3V3 gap at U5, WS_LVDS, WS_P, WS_T and WS_N.

Co-authored-by: fedurca <fedurca@users.noreply.github.com>
Parts:
- added JP_OE: OE, Connector_PinHeader_2.54mm:PinHeader_1x02_P2.54mm_Vertical, B.Cu at (46.8, 56.4)
- added JP_SCK: MODE, Connector_PinHeader_2.54mm:PinHeader_2x03_P2.54mm_Vertical, B.Cu at (25.4, 4.80)
- added JP_SD: MODE, Connector_PinHeader_2.54mm:PinHeader_2x03_P2.54mm_Vertical, B.Cu at (46.0, 17.8)
- added JP_SDN: SDN, Connector_PinHeader_2.54mm:PinHeader_1x03_P2.54mm_Vertical, B.Cu at (46.8, 46.0)
- added JP_TSCK: T, Connector_PinHeader_2.54mm:PinHeader_1x02_P2.54mm_Vertical, B.Cu at (2.50, 28.0)
- added JP_TWS: T, Connector_PinHeader_2.54mm:PinHeader_1x02_P2.54mm_Vertical, B.Cu at (2.50, 36.8)
- added JP_WS: MODE, Connector_PinHeader_2.54mm:PinHeader_2x03_P2.54mm_Vertical, B.Cu at (32.2, 4.80)
- added R_OE: 10k, Resistor_SMD:R_0603_1608Metric, B.Cu at (36.2, 16.8)
- added R_SD3: 100k, Resistor_SMD:R_0603_1608Metric, B.Cu at (36.2, 21.6)
Connections:
- J1 pad SH: (no net) -> GND
- R_SCK pad 2: SCK_N -> SCK_T
- R_WS pad 2: WS_N -> WS_T
- U2 pad 5: SCK_3V3 -> SCK_LVDS
- U3 pad 5: WS_3V3 -> WS_LVDS
- U4 pad 3: SD_P -> SD_Y
- U4 pad 4: SD_N -> SD_Z
- U5 pad 8: +3V3 -> OE
Routing:
- net WS: track 54.8 -> 284.9 mm, vias 3 -> 5
- net SCK_T: track 0.00 -> 215.3 mm
- net WS_3V3: track 23.0 -> 167.5 mm, vias 2 -> 3
- net SD_Y: track 0.00 -> 134.7 mm, vias 0 -> 2
- net SD_P: track 56.0 -> 159.0 mm
- net SCK: track 43.8 -> 118.6 mm
- net SD_Z: track 0.00 -> 68.7 mm
- net SD_N: track 38.5 -> 100.2 mm
- net SCK_P: track 71.9 -> 129.0 mm
- net SCK_3V3: track 88.7 -> 128.3 mm
- net SCK_LVDS: track 0.00 -> 36.0 mm, vias 0 -> 2
- net SD_3V3: track 33.9 -> 62.9 mm, vias 2 -> 4
- net SD: track 68.8 -> 81.0 mm
- net WS_N: track 66.2 -> 57.5 mm
- net +3V3: track 485.4 -> 479.5 mm
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Other:
- board text added: "1/2 SCK 3/6 WS 4/5 SD"
- board text added: "1V8 = kabel primo na T5848"
- board text added: "JP_T jen DIFF JP_OE jen 1V8"
- board text added: "het68 SAT rezim propojkou"
- board text added: "pin1 SV radek shora: DIFF 3V3 1V8"
- board text removed: "1/2 SCK 3/6 WS 4/5 SD 8x SK6812"
- board text removed: "het68 SAT v4 6L LVDS"

Commit message: Stand the RJ45 plugs upright and show the mode shunt.
The core and satellite jacks are a vertical 8P8C. The plug axis leaves
the board face instead of running off the edge. The docs and the v480
renders include the satellite mode headers. DRC has no shorts. Some
jack pins, and the tracks the new pad grid cut, are still open.

Co-authored-by: fedurca <fedurca@users.noreply.github.com>
Parts:
- J1: footprint het68:RJ45_RJHSE5380_het68 -> het68:RJ45_Vertical_het68
- moved J1 5.00 mm to (14.0, 11.0)
Routing:
- net WS_NJ: track 28.4 -> 45.0 mm
- net SD_PJ: track 53.2 -> 69.6 mm
- net SCK_NJ: track 23.2 -> 35.1 mm, vias 2 -> 3
- net SCK_PJ: track 27.9 -> 35.0 mm, vias 2 -> 3
- net SCK_P: track 129.0 -> 122.4 mm
- net WS_PJ: track 43.3 -> 47.0 mm
- net SD_NJ: track 53.7 -> 51.5 mm
- net SCK_T: track 215.3 -> 213.3 mm
- net 3V3_F: track 62.1 -> 60.6 mm, vias 5 -> 6
